File: spi.sch (EAGLE design)
At the start: 7 parts, among them IC2 25AA080SN, IC3 25AA080P, X1 2510-

Commit message: 25 серия использует so-8 в 200 mil
Parts:
- IC2: value 25AA080SN -> 25; device microchip:25AA080SN -> microchip:25
